File: kicad-mitsubishi-heavy-cns-ac-controller-v1/kicad-mitsubishi-heavy-cns-ac-controller-v1.kicad_pcb (KiCad board)
At the start: 2 copper layers, 42.7 x 48.8 mm, 30 parts, among them J3 USB_OTG, J4 Conn_01x05_Pin, SW1 SW_Push, SW2 SW_Push, U1 Si8641BB-B-IU, U2 AP2112K-3.3, U3 ESP32-C3-WROOM-02, U5 AOZ1282CI-1

Commit message: Add input capacitor, add text for cns
Parts:
- added C2: 100uF, Capacitor_Tantalum_SMD:CP_EIA-3528-12_Kemet-T_HandSolder, B.Cu at (75.3, 60.0)
Routing:
- net +3V3: track 107.3 -> 109.2 mm, vias 4 -> 6
Other:
- board text added: "12V"
- board text added: "GND"
- board text added: "MISO"
- board text added: "MOSI"
- board text added: "Mitsubishi Heavy CNS A/C ESP32 Controller v1.2"
- board text added: "SCK"
- board text removed: "Mitsubishi Heavy CNS A/C ESP32 Controller v1.0"

Commit message: Fix min trace spacing.
Was less than 0.1mm even though it was the same track.
Routing:
- net +3V3: track 109.2 -> 109.7 mm
Other:
- board text added: "Mitsubishi Heavy CNS A/C ESP32 Controller v1.3"
- board text removed: "Mitsubishi Heavy CNS A/C ESP32 Controller v1.2"
Changed lines of the file:
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@@
 		)
 	)
-	(gr_text "Mitsubishi Heavy CNS A/C\nESP32 Controller v1.2"
+	(gr_text "Mitsubishi Heavy CNS A/C\nESP32 Controller v1.3"
 		(at 95.025 94.3 0)
 		(layer "F.SilkS")
@@
 	)
 	(segment
-		(start 92.0875 78.028812)
-		(end 91.731312 78.385)
+		(start 111.5 51.575)
+		(end 107.75 51.575)
+		(width 0.25)
+		(layer "F.Cu")
+		(net 4)
+	)
+	(segment
+		(start 91.762499 74.575)
+		(end 92.775 75.587501)
+		(width 0.25)
+		(layer "F.Cu")
+		(net 4)
+	)
+	(segment
+		(start 107.75 51.575)
+		(end 107.725 51.55)
+		(width 0.25)
+		(layer "F.Cu")
+		(net 4)
+	)
+	(segment
+		(start 86.085 64.01)
+		(end 86.085 66.55)
+		(width 1)
+		(layer "F.Cu")
+		(net 4)
+	)
+	(segment
+		(start 78.325 58)
+		(end 74.95 58)
+		(width 1)
+		(layer "F.Cu")
+		(net 4)
+	)
+	(segment
+		(start 80.375 58.15)
+		(end 78.575 58.15)
+		(width 0.25)
+		(layer "F.Cu")
+		(net 4)
+	)
+	(segment
+		(start 87.85 78.4)
+		(end 88.5 78.4)
+		(width 0.25)
+		(layer "F.Cu")
+		(net 4)
+	)
+	(segment
+		(start 78.525 58.2)
+		(end 80.275 58.2)
+		(width 1)
+		(layer "F.Cu")
+		(net 4)
+	)
+	(segment
+		(start 88.515 78.385)
+		(end 90.95 78.385)
+		(width 0.25)
+		(layer "F.Cu")
+		(net 4)
+	)
+	(segment
+		(start 78.525 58.2)
+		(end 78.325 58)
+		(width 1)
+		(layer "F.Cu")
+		(net 4)
+	)
+	(segment
+		(start 92.775 75.587501)
+		(end 92.775 77.341312)
+		(width 0.25)
+		(layer "F.Cu")
+		(net 4)
+	)
+	(segment
+		(start 86.085 66.55)
+		(end 92.775 73.24)
+		(width 1)
+		(layer "F.Cu")
+		(net 4)
+	)
+	(segment
+		(start 107.725 51.55)
+		(end 102.175 57.1)
+		(width 0.25)
+		(layer "F.Cu")
+		(net 4)
+	)
+	(segment
+		(start 102.175 57.1)
+		(end 102.175 61.15)
 		(width 0.25)
 		(layer "F.Cu")
@@
 	)
 	(segment
-		(start 111.5 51.575)
-		(end 107.75 51.575)
-		(width 0.25)
-		(layer "F.Cu")
-		(net 4)
-	)
-	(segment
-		(start 107.75 51.575)
+		(start 78.575 58.15)
+		(end 78.525 58.2)
+		(width 0.25)
+		(layer "F.Cu")
+		(net 4)
+	)
+	(segment
+		(start 74.25 58.7)
+		(end 74.25 59.175)
+		(width 1)
+		(layer "F.Cu")
+		(net 4)
+	)
+	(segment
+		(start 92.775 73.24)
+		(end 92.775 82.3)
+		(width 1)
+		(layer "F.Cu")
+		(net 4)
+	)
+	(segment
+		(start 105.875 51.575)
+		(end 107.7 51.575)
+		(width 0.25)
+		(layer "F.Cu")
+		(net 4)
+	)
+	(segment
+		(start 107.7 51.575)
 		(end 107.725 51.55)
 		(width 0.25)
@@
 	)
 	(segment
-		(start 86.085 64.01)
-		(end 86.085 66.55)
-		(width 1)
-		(layer "F.Cu")
-		(net 4)
-	)
-	(segment
-		(start 78.325 58)
-		(end 74.95 58)
-		(width 1)
-		(layer "F.Cu")
-		(net 4)
-	)
-	(segment
-		(start 80.375 58.15)
-		(end 78.575 58.15)
-		(width 0.25)
-		(layer "F.Cu")
-		(net 4)
-	)
-	(segment
-		(start 87.85 78.4)
-		(end 88.5 78.4)
-		(width 0.25)
-		(layer "F.Cu")
-		(net 4)
-	)
-	(segment
-		(start 92.0875 74.900001)
-		(end 92.0875 78.028812)
-		(width 0.25)
-		(layer "F.Cu")
-		(net 4)
-	)
-	(segment
-		(start 78.525 58.2)
-		(end 80.275 58.2)
+		(start 80.275 58.2)
+		(end 86.085 64.01)
+		(width 1)
+		(layer "F.Cu")
+		(net 4)
+	)
+	(segment
+		(start 92.775 77.341312)
+		(end 91.731312 78.385)
+		(width 0.25)
+		(layer "F.Cu")
+		(net 4)
+	)
+	(segment
+		(start 74.95 58)
+		(end 74.25 58.7)
 		(width 1)
 		(layer "F.Cu")
@@
 		(layer "F.Cu")
 		(net 4)
-	)
-	(segment
-		(start 88.515 78.385)
-		(end 90.95 78.385)
-		(width 0.25)
-		(layer "F.Cu")
-		(net 4)
-	)
-	(segment
-		(start 78.525 58.2)
-		(end 78.325 58)
-		(width 1)
-		(layer "F.Cu")
-		(net 4)
-	)
-	(segment
-		(start 86.085 66.55)
-		(end 92.775 73.24)
-		(width 1)
-		(layer "F.Cu")
-		(net 4)
-	)
-	(segment
-		(start 107.725 51.55)
-		(end 102.175 57.1)
-		(width 0.25)
-		(layer "F.Cu")
-		(net 4)
-	)
-	(segment
-		(start 102.175 57.1)
-		(end 102.175 61.15)
-		(width 0.25)
-		(layer "F.Cu")
-		(net 4)
-	)
-	(segment
-		(start 78.575 58.15)
-		(end 78.525 58.2)
-		(width 0.25)
-		(layer "F.Cu")
-		(net 4)
-	)
-	(segment
-		(start 74.25 58.7)
-		(end 74.25 59.175)
-		(width 1)
-		(layer "F.Cu")
-		(net 4)
-	)
-	(segment
-		(start 91.762499 74.575)
-		(end 92.0875 74.900001)
-		(width 0.25)
-		(layer "F.Cu")
-		(net 4)
-	)
-	(segment
-		(start 92.775 73.24)
-		(end 92.775 82.3)
-		(width 1)
-		(layer "F.Cu")
-		(net 4)
-	)
-	(segment
-		(start 105.875 51.575)
-		(end 107.7 51.575)
-		(width 0.25)
-		(layer "F.Cu")
-		(net 4)
-	)
-	(segment
-		(start 107.7 51.575)
-		(end 107.725 51.55)
-		(width 0.25)
-		(layer "F.Cu")
-		(net 4)
-	)
-	(segment
-		(start 80.275 58.2)
-		(end 86.085 64.01)
-		(width 1)
-		(layer "F.Cu")
-		(net 4)
-	)
-	(segment
-		(start 74.95 58)
-		(end 74.25 58.7)
-		(width 1)
-		(layer "F.Cu")
-		(net 4)

Commit message: Fix digital isolator to be tied to 5v not 12v
Connections:
- U1 pad 10: +12V -> +5V
- U1 pad 16: +12V -> +5V
Routing:
- net +12V: track 61.9 -> 38.9 mm
- net +5V: track 36.9 -> 52.3 mm
Other:
- board text added: "Mitsubishi Heavy CNS A/C ESP32 Controller v1.4"
- board text removed: "Mitsubishi Heavy CNS A/C ESP32 Controller v1.3"
Changed lines of the file:
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@@
 			(layers "F.Cu" "F.Mask" "F.Paste")
 			(roundrect_rratio 0.25)
-			(net 1 "+12V")
+			(net 22 "+5V")
 			(pinfunction "EN2")
 			(pintype "input")
@@
 			(layers "F.Cu" "F.Mask" "F.Paste")
 			(roundrect_rratio 0.25)
-			(net 1 "+12V")
+			(net 22 "+5V")
 			(pinfunction "VDD2")
 			(pintype "power_in")
@@
 		)
 	)
-	(gr_text "Mitsubishi Heavy CNS A/C\nESP32 Controller v1.3"
+	(gr_text "Mitsubishi Heavy CNS A/C\nESP32 Controller v1.4"
 		(at 95.025 94.3 0)
 		(layer "F.SilkS")
@@
 	)
 	(segment
-		(start 95.412501 78.385)
-		(end 96.225 78.385)
-		(width 0.25)
-		(layer "F.Cu")
-		(net 1)
-	)
-	(segment
 		(start 111.9 78.25)
 		(end 113 78.25)
@@
 	)
 	(segment
-		(start 95.0875 74.900001)
-		(end 95.0875 78.059999)
-		(width 0.25)
-		(layer "F.Cu")
-		(net 1)
-	)
-	(segment
-		(start 108.025 74.375)
-		(end 111.9 78.25)
-		(width 0.25)
-		(layer "F.Cu")
-		(net 1)
-	)
-	(segment
-		(start 95.412501 74.575)
-		(end 95.0875 74.900001)
-		(width 0.25)
-		(layer "F.Cu")
-		(net 1)
-	)
-	(segment
-		(start 96.425 74.375)
-		(end 108.025 74.375)
-		(width 0.25)
-		(layer "F.Cu")
-		(net 1)
-	)
-	(segment
-		(start 96.225 74.575)
-		(end 96.425 74.375)
-		(width 0.25)
-		(layer "F.Cu")
-		(net 1)
-	)
-	(segment
-		(start 95.0875 78.059999)
-		(end 95.412501 78.385)
-		(width 0.25)
-		(layer "F.Cu")
-		(net 1)
-	)
-	(segment
-		(start 96.225 74.575)
-		(end 95.412501 74.575)
-		(width 0.25)
-		(layer "F.Cu")
-		(net 1)
-	)
-	(segment
 		(start 107.975 85.725)
 		(end 108.6375 86.3875)
@@
 	)
 	(segment
-		(start 96.225 75.21)
-		(end 98.585 75.21)
+		(start 98.51 75.21)
+		(end 98.65 75.35)
 		(width 0.25)
 		(layer "F.Cu")
@@
 	)
 	(segment
-		(start 98.585 75.21)
-		(end 98.65 75.275)
+		(start 96.225 75.21)
+		(end 98.51 75.21)
 		(width 0.25)
 		(layer "F.Cu")
@@
 	)
 	(via
-		(at 98.65 75.275)
+		(at 98.65 75.35)
 		(size 0.8)
 		(drill 0.4)
@@
 	)
 	(segment
-		(start 98.122588 76.48)
-		(end 98.142588 76.5)
+		(start 98.142588 76.575)
+		(end 106.245 76.575)
 		(width 0.25)
 		(layer "F.Cu")
@@
 	)
 	(segment
-		(start 98.142588 76.5)
-		(end 106.17 76.5)
+		(start 96.225 76.48)
+		(end 98.047588 76.48)
 		(width 0.25)
 		(layer "F.Cu")
@@
 	)
 	(segment
-		(start 96.225 76.48)
-		(end 98.122588 76.48)
+		(start 98.047588 76.48)
+		(end 98.142588 76.575)
 		(width 0.25)
 		(layer "F.Cu")
@@
 	)
 	(segment
-		(start 106.17 76.5)
+		(start 106.245 76.575)
 		(end 113 83.33)
 		(width 0.25)
@@
 	(segment
 		(start 96.225 75.845)
-		(end 98.123984 75.845)
+		(end 98.048984 75.845)
 		(width 0.25)
 		(layer "F.Cu")
@@
 	)
 	(segment
-		(start 108.26 76.05)
-		(end 113 80.79)
+		(start 98.328984 76.125)
+		(end 108.335 76.125)
 		(width 0.25)
 		(layer "F.Cu")
@@
 	)
 	(segment
-		(start 98.123984 75.845)
-		(end 98.328984 76.05)
+		(start 108.335 76.125)
+		(end 113 80.79)
 		(width 0.25)
 		(layer "F.Cu")
@@
 	)
 	(segment
-		(start 98.328984 76.05)
-		(end 108.26 76.05)
+		(start 98.048984 75.845)
+		(end 98.328984 76.125)
 		(width 0.25)
 		(layer "F.Cu")
@@
 		(width 0.25)
 		(layer "F.Cu")
+		(net 22)
+	)
+	(segment
+		(start 95.412501 78.385)
+		(end 96.225 78.385)
+		(width 0.25)
+		(layer "F.Cu")
+		(net 22)
+	)
+	(segment
+		(start 95.0875 74.900001)
+		(end 95.0875 78.059999)
+		(width 0.25)
+		(layer "F.Cu")
+		(net 22)
+	)
+	(segment
+		(start 103.65 74.575)
+		(end 105.275 72.95)
+		(width 0.25)
+		(layer "F.Cu")
+		(net 22)
+	)
+	(segment
+		(start 95.412501 74.575)
+		(end 95.0875 74.900001)
+		(width 0.25)
+		(layer "F.Cu")
+		(net 22)
+	)
+	(segment
+		(start 96.225 74.575)
+		(end 103.65 74.575)
+		(width 0.25)
+		(layer "F.Cu")
+		(net 22)
+	)
+	(segment
+		(start 95.0875 78.059999)
+		(end 95.412501 78.385)
+		(width 0.25)
+		(layer "F.Cu")
+		(net 22)
+	)
+	(segment
+		(start 96.225 74.575)
+		(end 95.412501 74.575)
+		(width 0.25)
+		(layer "F.Cu")

Commit message: Fix 5v to gnd issue. Update resistors for buck converter.
Other:
- board text added: "Mitsubishi Heavy CNS A/C ESP32 Controller v1.5"
- board text removed: "Mitsubishi Heavy CNS A/C ESP32 Controller v1.4"
Changed lines of the file:
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@@
 		)
 	)
-	(gr_arc
-		(start 73.025 47)
-		(mid 73.317893 46.292893)
-		(end 74.025 46)
-		(stroke
-			(width 0.1)
-			(type default)
-		)
-		(layer "Edge.Cuts")
-	)
 	(gr_line
-		(start 73.025 93.8)
-		(end 73.025 47)
-		(stroke
-			(width 0.1)
-			(type default)
-		)
-		(layer "Edge.Cuts")
-	)
-	(gr_line
-		(start 74.025 46)
-		(end 114.725 46)
+		(start 115.725 47)
+		(end 115.725 93.8)
 		(stroke
 			(width 0.1)
@@
 		(mid 73.317893 94.507107)
 		(end 73.025 93.8)
+		(stroke
+			(width 0.1)
+			(type default)
+		)
+		(layer "Edge.Cuts")
+	)
+	(gr_arc
+		(start 115.725 93.8)
+		(mid 115.432107 94.507107)
+		(end 114.725 94.8)
 		(stroke
 			(width 0.1)
@@
 	)
 	(gr_line
-		(start 115.725 47)
-		(end 115.725 93.8)
+		(start 74.025 46)
+		(end 114.725 46)
+		(stroke
+			(width 0.1)
+			(type default)
+		)
+		(layer "Edge.Cuts")
+	)
+	(gr_line
+		(start 73.025 93.8)
+		(end 73.025 47)
 		(stroke
 			(width 0.1)
@@
 	)
 	(gr_arc
-		(start 115.725 93.8)
-		(mid 115.432107 94.507107)
-		(end 114.725 94.8)
+		(start 73.025 47)
+		(mid 73.317893 46.292893)
+		(end 74.025 46)
 		(stroke
 			(width 0.1)
@@
 		)
 	)
-	(gr_text "Mitsubishi Heavy CNS A/C\nESP32 Controller v1.4"
+	(gr_text "Mitsubishi Heavy CNS A/C\nESP32 Controller v1.5"
 		(at 95.025 94.3 0)
 		(layer "F.SilkS")
@@
 		)
 	)
-	(gr_text "MOSI"
-		(at 107.55 83.825 0)
+	(gr_text "MISO"
+		(at 107.575 86.45 0)
 		(layer "F.SilkS")
 		(effects
@@
 		)
 	)
-	(gr_text "MISO"
-		(at 107.575 86.45 0)
+	(gr_text "12V"
+		(at 108.225 78.775 0)
 		(layer "F.SilkS")
 		(effects
@@
 		)
 	)
-	(gr_text "12V"
-		(at 108.225 78.775 0)
+	(gr_text "SCK"
+		(at 108.25 81.325 0)
 		(layer "F.SilkS")
 		(effects
@@
 		)
 	)
-	(gr_text "SCK"
-		(at 108.25 81.325 0)
+	(gr_text "MOSI"
+		(at 107.55 83.825 0)
 		(layer "F.SilkS")
 		(effects
